File: kicad-setting-boards/jlcpcb-4Layer-JLC04161H-2116D/jlcpcb-4Layer-JLC04161H-2116D.kicad_pcb (KiCad board)
At the start: 4 copper layers, 0 parts

Commit message: adding outline for docker example
Other:
- board outline added: 101.6 x 35.6 mm
Changed lines of the file:
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@@
 		(layer "Dwgs.User")
+	)
+	(gr_rect
+		(start 81.28 88.9)
+		(end 182.88 124.46)
+		(stroke
+			(width 0.05)
+			(type default)
+		)
+		(fill none)
+		(layer "Edge.Cuts")
 	)
 	(gr_text "0 mm"
